Commit message: feat(gate_config_9): per-env trajectory metrics + W&B obs-grad + curriculum
Environment/task (gate navigation)
- Track per-env episode state: spawn pos, gate center at spawn, last pos, path length
  accumulation, step counter, min distance to gate center, first-cross center/height
  offsets, and last-position at episode end.
- Use true gate center (z-corrected) for per-step gate distance and per-episode
  min_gate_distance so values can approach 0 on perfect center passes.
- Fix info propagation across resets: stash infos before reset and return the stashed
  dict on the next get_return_tuple() to avoid losing episode-end metrics.

W&B logging (worker + learner)
- Worker: Log per-episode counts (successes/crashes/timeouts), cumulative totals
  (curriculum/total_*), current curriculum snapshot (level/progress), gate/camera
  alignment metrics, curriculum snapshot details (env totals, camera noise/dropout,
  freeze/blank components, camera angles, state noise), and trajectory end metrics
  (last_position_x/y/z, last_center_distance) under episode_extra_stats/*.
- Learner: Force enhanced path; mirror obs-grad keys into episode_extra_stats/obs_grad/*;
  compute camera/state shares (+ pct), log per-slice magnitudes and percentages; cache
  last tracker outputs; add explicit, every-step wandb.log for obs-grad.

Curriculum policy
- Window: 256 instances; thresholds: increase @ 0.6, decrease @ 0.25 (decrease enabled).
- Add cooldown_windows=2 via internal cooldown counter to prevent oscillation; include
  cooldown status in printed curriculum summary.

URDF fixes
- Gates: normalize frame thickness to 0.110 m in gate_scale_050.urdf and gate_scale_046.urdf
  (visual + collision).
- Obstacles: adjust placeholder box dims to correct volumes (e.g., ~0.908 scale for 2x,
  ~0.794 for 1x/1.5x variants) across rectangular/trapezoid/triangular assets.

Repo hygiene
- Add repo-root .gitignore to exclude python caches, checkpoints (*.pth), training dirs,
  W&B run data, tensorboard events, logs, and generated GIFs.

Notes
- Trajectory metrics now robust to vectorized async resets; center-corrected distances and
  path efficiency computed per env; expanded episode_extra_stats improves analysis and W&B
  visibility; curriculum is more stable with decrease+cooldown.

File: resources/models/environment_assets/gates/gate_scale_046.urdf (robot description, URDF)
Before this commit: robot gate_scale_046, 5 links, 4 joints
Links:
- link left_post: geometry collision box size=0.110 0.110 1.150; visual box size=0.110 0.110 1.150
- link top_bar: geometry collision box size=0.110 1.242 0.110; visual box size=0.110 1.242 0.110

File: resources/models/environment_assets/gates/gate_scale_050.urdf (robot description, URDF)
Before this commit: robot gate_scale_050, 5 links, 4 joints
Links:
- link left_post: geometry collision box size=0.110 0.110 1.250; visual box size=0.110 0.110 1.250
- link top_bar: geometry collision box size=0.110 1.350 0.110; visual box size=0.110 1.350 0.110

File: resources/models/environment_assets/objects_gate/rectangular_box_1_5x.urdf (robot description, URDF)
Before this commit: robot rectangular_box, 1 links, 0 joints
Links:
- link base_link: geometry collision box size=0.954 0.477 0.716; visual box size=0.954 0.477 0.716

File: resources/models/environment_assets/objects_gate/rectangular_box_1x.urdf (robot description, URDF)
Before this commit: robot rectangular_box, 1 links, 0 joints
Links:
- link base_link: geometry collision box size=0.636 0.318 0.477; visual box size=0.636 0.318 0.477

File: resources/models/environment_assets/objects_gate/rectangular_box_2x.urdf (robot description, URDF)
Before this commit: robot rectangular_box, 1 links, 0 joints
Links:
- link base_link: geometry collision box size=1.271 0.636 0.954; visual box size=1.271 0.636 0.954

File: resources/models/environment_assets/objects_gate/trapezoid_1_5x.urdf (robot description, URDF)
Before this commit: robot trapezoid, 1 links, 0 joints
Links:
- link base_link: geometry collision box size=1.429 0.952 0.476; visual box size=1.429 0.952 0.476

File: resources/models/environment_assets/objects_gate/trapezoid_1x.urdf (robot description, URDF)
Before this commit: robot trapezoid, 1 links, 0 joints
Links:
- link base_link: geometry collision box size=0.952 0.635 0.318; visual box size=0.952 0.635 0.318

File: resources/models/environment_assets/objects_gate/trapezoid_2x.urdf (robot description, URDF)
Before this commit: robot trapezoid, 1 links, 0 joints
Links:
- link base_link: geometry collision box size=1.732 1.155 0.578; visual box size=1.732 1.155 0.578

File: resources/models/environment_assets/objects_gate/triangular_prism_2x.urdf (robot description, URDF)
Before this commit: robot triangular_prism, 1 links, 0 joints
Links:
- link base_link: geometry collision box size=1.818 0.545 1.091; visual box size=1.818 0.545 1.091

Commit message: advanced ablation studies config9 21/08

File: resources/models/environment_assets/gates/gate_scale_046.urdf (robot description, URDF)
Before this commit: robot gate_scale_046, 5 links, 4 joints
Links:
- link right_post: geometry collision box size=0.110 0.110 1.150; visual box size=0.110 0.110 1.150

File: resources/models/environment_assets/gates/gate_scale_050.urdf (robot description, URDF)
Before this commit: robot gate_scale_050, 5 links, 4 joints
Links:
- link right_post: geometry collision box size=0.110 0.110 1.250; visual box size=0.110 0.110 1.250
