Commit message: Untrack static_frames_480x270/val images and ignore

File: resources/models/environment_assets/objects_gate/cylinder_2x.urdf (robot description, URDF)
Before this commit: robot cylinder, 1 links, 0 joints
Links:
- link base_link: geometry collision cylinder length=1.587 radius=0.317; visual cylinder length=1.587 radius=0.317

File: resources/models/environment_assets/objects_gate/rectangular_box_2x.urdf (robot description, URDF)
Before this commit: robot rectangular_box, 1 links, 0 joints
Links:
- link base_link: geometry collision box size=1.009 0.505 0.757; visual box size=1.009 0.505 0.757

File: resources/models/environment_assets/objects_gate/small_cube_2x.urdf (robot description, URDF)
Before this commit: robot box, 1 links, 0 joints
Links:
- link base_link: geometry collision box size=0.635 0.635 0.635; visual box size=0.635 0.635 0.635

File: resources/models/environment_assets/objects_gate/sphere_2x.urdf (robot description, URDF)
Before this commit: robot sphere, 1 links, 0 joints
Links:
- link base_link: geometry collision sphere radius=0.476; visual sphere radius=0.476

File: resources/models/environment_assets/objects_gate/trapezoid_1_5x.urdf (robot description, URDF)
Before this commit: robot trapezoid, 1 links, 0 joints
Links:
- link base_link: geometry collision box size=1.134 0.756 0.378; visual box size=1.134 0.756 0.378

File: resources/models/environment_assets/objects_gate/trapezoid_2x.urdf (robot description, URDF)
Before this commit: robot trapezoid, 1 links, 0 joints
Links:
- link base_link: geometry collision box size=1.375 0.917 0.459; visual box size=1.375 0.917 0.459

File: resources/models/environment_assets/objects_gate/triangular_prism_1_5x.urdf (robot description, URDF)
Before this commit: robot triangular_prism, 1 links, 0 joints
Links:
- link base_link: geometry collision box size=1.191 0.357 0.714; visual box size=1.191 0.357 0.714

File: resources/models/environment_assets/objects_gate/triangular_prism_2x.urdf (robot description, URDF)
Before this commit: robot triangular_prism, 1 links, 0 joints
Links:
- link base_link: geometry collision box size=1.443 0.433 0.866; visual box size=1.443 0.433 0.866
